File: circuit/circuit.kicad_sch (KiCad schematic)
At the start: 0 parts

Commit message: 1
Parts:
- added C1, C12, C14, C17, C20, C31, C37, C38, C5: 10uf, Capacitor_SMD:C_0603_1608Metric, symbol Device:C
- added C10, C11, C16, C18, C2, C21, C26, C27, C28, C30, C32, C34, C36, C4, C6, C8, C9: 0.1uf, Capacitor_SMD:C_0603_1608Metric, symbol Device:C
- added C13, C7: 18pf, Capacitor_SMD:C_0603_1608Metric, symbol Device:C
- added C15: 1uf, Capacitor_SMD:C_0603_1608Metric, symbol Device:C
- added C19: 4.7nf, Capacitor_SMD:C_0603_1608Metric, symbol Device:C
- added C23, C35: 0.1uf, Capacitor_SMD:C_0805_2012Metric, symbol Device:C
- added C24: 0.47uf, Capacitor_SMD:C_0603_1608Metric, symbol Device:C
- added C25: 1uf, Capacitor_THT:C_Axial_L12.0mm_D6.5mm_P20.00mm_Horizontal, symbol Device:C
- added C29: 0.01uf, Capacitor_SMD:C_0603_1608Metric, symbol Device:C
- added C3: 220uf, Capacitor_THT:CP_Radial_D6.3mm_P2.50mm, symbol Device:C_Polarized_US
- added D1: LED, LED_SMD:LED_0603_1608Metric, symbol Device:LED
- added D2, D5: 1N5819WS, Diode_SMD:D_SOD-323_HandSoldering, symbol Diode:1N5819WS
- added D3: B340A, Diode_SMD:D_SMA, symbol Diode:B340
- added D4: LED, LED_SMD:LED_0805_2012Metric_Pad1.15x1.40mm_HandSolder, symbol Device:LED
- added D6, D7, D8, D9: 1N4148W, Diode_SMD:D_SOD-123, symbol Diode:1N4148W
- added ENA1: EN, TestPoint:TestPoint_Pad_D1.0mm, symbol Connector:TestPoint
- added FB2: 600Ω@100MHz, Resistor_SMD:R_0603_1608Metric, symbol Device:FerriteBead_Small
- added H1, H2, H3, H5: MountingHole, MountingHole:MountingHole_2.2mm_M2_ISO7380_Pad, symbol Mechanical:MountingHole
- added J1: Barrel_Jack_Switch, Connector_BarrelJack:BarrelJack_Horizontal, symbol Connector:Barrel_Jack_Switch
- added J2: Conn_01x04, Connector_PinHeader_2.54mm:PinHeader_1x04_P2.54mm_Vertical, symbol Connector_Generic:Conn_01x04
- added J4: AudioJack3_SwitchTR, Connector_Audio:Jack_3.5mm_Lumberg_1503_02_Horizontal, symbol Connector_Audio:AudioJack3_SwitchTR
- added J5: Conn_01x05, Connector_PinHeader_2.54mm:PinHeader_1x05_P2.54mm_Vertical, symbol Connector_Generic:Conn_01x05
- added L1: 15uh, Inductor_SMD:L_Changjiang_FXL0630, symbol Device:L_Iron
- added L2, L3: 22uh, Inductor_SMD:L_Changjiang_FXL0630, symbol Device:L_Iron
- added LS1: 8R, TerminalBlock:TerminalBlock_MaiXu_MX126-5.0-02P_1x02_P5.00mm, symbol Device:Speaker
- added Q1, Q2, Q3, Q4: IRLR7843, Package_TO_SOT_SMD:TO-252-2, symbol Simulation_SPICE:NMOS
- added R1: 2K, Resistor_SMD:R_0603_1608Metric, symbol Device:R
- added R10, R22: 100R, Resistor_SMD:R_0603_1608Metric, symbol Device:R
- added R11, R3: 1k, Resistor_SMD:R_0603_1608Metric, symbol Device:R
- added R12, R13, R20, R21: 20R, Resistor_SMD:R_0603_1608Metric, symbol Device:R
- added R14, R17, R2: 0R, Resistor_SMD:R_0603_1608Metric, symbol Device:R
- added R15, R19: 33R, Resistor_SMD:R_0603_1608Metric, symbol Device:R
- added R16, R28, R29, R31, R32, R33, R4, R5, R6, R7, R8: 10k, Resistor_SMD:R_0603_1608Metric, symbol Device:R
- added R18, R23, R24, R25: 10K, Resistor_SMD:R_0603_1608Metric, symbol Device:R
- added R26: 3.24K, Resistor_SMD:R_0603_1608Metric, symbol Device:R
- added R27: 12k, Resistor_SMD:R_0603_1608Metric, symbol Device:R
- added R30: 2k, Resistor_SMD:R_0603_1608Metric, symbol Device:R
- added R9: 1R, Resistor_SMD:R_0603_1608Metric, symbol Device:R
- added SW1: SW_Nidec_CAS-120A1, Button_Switch_SMD:SW_SPDT_CK_JS102011SAQN, symbol Switch:SW_Nidec_CAS-120A1
- added SW2: SW_SPST, Button_Switch_SMD:SW_Tactile_SPST_NO_Straight_CK_PTS636Sx25SMTRLFS, symbol Switch:SW_SPST
- added U1: AMS1117-3.3, Package_TO_SOT_SMD:SOT-223-3_TabPin2, symbol Regulator_Linear:AMS1117-3.3
- added U2: TPS5430DDA, Package_SO:TI_SO-PowerPAD-8_ThermalVias, symbol Regulator_Switching:TPS5430DDA
- added U3: TLV9062, Package_SO:SOIC-8_5.3x5.3mm_P1.27mm, symbol Amplifier_Operational:TLV9062
- added U4, U6: IR2104, Package_SO:PowerIntegrations_SO-8, symbol Driver_FET:IR2104
- added U5: STM32G431CBTx, Package_QFP:LQFP-48_7x7mm_P0.5mm, symbol MCU_ST_STM32G4:STM32G431CBTx
- added Y2: Crystal_GND24, Crystal:Crystal_SMD_EuroQuartz_MT-4Pin_3.2x2.5mm, symbol Device:Crystal_GND24
Connections:
- new net: R19.2, U6.2 (IN)
- new net: R18.1, U5.45 (PB8)
- new net: C35.2, L3.1, Q3.3 (S), Q4.1 (D), R32.1, U6.6 (VS)
- new net: D9.2 (A), Q4.2 (G), R21.2, R33.2
- new net: C16.1, C17.1, R7.2, R8.1, U3.3 (+)
- new net: J4.R, R5.1
- new net: C15.2, R4.2, R5.2
- new net: C25.1, L2.2, LS1.1, R9.2
- new net: C24.2, C25.2, L3.2, LS1.2
- new net: C23.2, L2.1, Q1.3 (S), Q2.1 (D), R29.1, U4.6 (VS)
- new net: D7.2 (A), Q2.2 (G), R13.2, R31.2
- new net: R10.2, R23.2, U4.3 (~{SD})
- new net: C35.1, D5.1 (K), U6.8 (VB)
- new net: C28.1, FB2.2, R14.1
- new net: D9.1 (K), R21.1, U6.5 (LO)
- new net: R22.2, R24.2, U6.3 (~{SD})
- new net: C29.2, D3.1 (K), L1.1, U2.8 (PH)
- new net: C29.1, U2.1 (BOOT)
- new net: D4.2 (A), R30.2
- new net: D8.1 (K), R20.1, U6.7 (HO)
- new net: D8.2 (A), Q3.2 (G), R20.2, R32.2
- new net: R11.1, R27.2, U3.7
- new net: C15.1, R6.2, U3.5 (+)
- new net: J1.1, SW1.2 (B)
- new net: R3.1, U3.1, U3.2 (-)
- new net: D7.1 (K), R13.1, U4.5 (LO)
- new net: J4.T, R4.1
- new net: R25.2, R26.1, U2.4 (VSENSE)
- new net: C23.1, D2.1 (K), U4.8 (VB)
- new net: C24.1, R9.1
- new net: R27.1, R28.2, U3.6 (-)
- new net: R15.2, U4.2 (IN)
- new net: D1.2 (A), R1.2
- new net: D6.2 (A), Q1.2 (G), R12.2, R29.2
- new net: ENA1.1, U2.5 (EN)
- new net: D6.1 (K), R12.1, U4.7 (HO)
- new net +12V: C12.1, C20.1, C21.1, C27.1, C30.1, C31.1, C32.1, C36.1, C37.1, C38.1, D2.2 (A), D5.2 (A), Q1.1 (D), Q3.1 (D), SW1.3 (A), U2.7 (VIN), U4.1 (VCC), U6.1 (VCC)
- new net +3V3: C10.1, C11.1, C14.1, C18.1, C6.1, C8.1, C9.1, J2.1 (Pin_1), J5.1 (Pin_1), R1.1, R14.2, R16.1, R30.1, R7.1, U1.2 (VO), U3.8 (V+), U5.1 (VBAT), U5.24 (VDD), U5.36 (VDD), U5.48 (VDD)
- new net +5V: C3.1, C4.1, C5.1, L1.2, R25.1, U1.3 (VI)
- new net ADC_in: C19.1, R11.2, U5.8 (PA0)
- new net AGND: C1.2, C16.2, C17.2, C18.2, C19.2, C2.2, C28.2, C34.2, J4.S, R17.1, R8.2, U3.4 (V-), U5.19 (VSSA)
- new net GND: C10.2, C11.2, C13.2, C14.2, C26.1, C4.2, C5.2, C6.2, C7.2, C8.2, C9.2, D1.1 (K), J2.4 (Pin_4), J5.5 (Pin_5), R17.2, R18.2, R2.2, SW2.2 (B), U1.1 (GND), U5.23 (VSS), U5.35 (VSS), U5.47 (VSS), Y2.2 (G), Y2.4 (G)
- new net KEY: J5.2 (Pin_2), U5.43 (PB6)
- new net NRST: C26.2, R16.2, SW2.1 (A), U5.7 (PG10)
- new net OSC_N: C13.1, U5.6 (PF1), Y2.3
- new net OSC_P: C7.1, U5.5 (PF0), Y2.1
- new net PC13: D4.1 (K), U5.2 (PC13)
- new net PGND: C12.2, C20.2, C21.2, C27.2, C3.2, C30.2, C31.2, C32.2, C36.2, C37.2, C38.2, D3.2 (A), J1.2, Q2.3 (S), Q4.3 (S), R2.1, R23.1, R24.1, R26.2, R31.1, R33.1, U2.6 (GND), U2.9 (GNDPAD), U4.4 (COM), U6.4 (COM)
- new net S1: J5.4 (Pin_4), U5.41 (PB4)
- new net S2: J5.3 (Pin_3), U5.42 (PB5)
- new net SD_A: R10.1, U5.32 (PA10)
- new net SD_B: R22.1, U5.29 (PB15)
- new net SWCLK: J2.3 (Pin_3), U5.38 (PA14)
- new net SWDIO: J2.2 (Pin_2), U5.37 (PA13)
- new net TIM1_CH1: R19.1, U5.30 (PA8)
- new net TIM1_CH2: R15.1, U5.31 (PA9)
- new net VCCA+3V3: C34.1, FB2.1, U5.20 (VREF+), U5.21 (VDDA)
- new net VREF: C1.1, C2.1, R28.1, R3.2, R6.1
- no-connect marks 0 -> 27
Other:
- note added: "MCU"
- note added: "MCU指示灯"
- note added: "下载调试电路"
- note added: "地隔离"
- note added: "复位电路"
- note added: "晶振"
- note added: "滤波电容"
- note added: "电源指示灯"
- note added: "电源管理"
- note added: "编码器"
- note added: "音频输入"
- note added: "音频输出"
